File: kicad/TinyRotaryPCB.kicad_sch (KiCad schematic)
At the start: 5 parts, among them J1 Conn_01x05_Pin, SW1 RotaryEncoder_Switch

Commit message: Update KiCad project, horizontal pin header
Parts:
- J1: footprint Connector_PinHeader_2.54mm:PinHeader_1x05_P2.54mm_Vertical -> PinHeader_1x05_P2.54mm_H_W_S:PinHeader_1x05_P2.54mm_Horizontal_Without_Silkscreen
Changed lines of the file:
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@@
 			)
 		)
-		(property "Footprint" "Connector_PinHeader_2.54mm:PinHeader_1x05_P2.54mm_Vertical"
+		(property "Footprint" "PinHeader_1x05_P2.54mm_H_W_S:PinHeader_1x05_P2.54mm_Horizontal_Without_Silkscreen"
 			(at 109.22 92.71 0)
 			(effects
@@
 			)
 		)
-		(property "Description" "Generic connector, single row, 01x05, script generated"
+		(property "Description" "Generic connector, single row, 01x05, without silkscreen (minimal)"
 			(at 109.22 92.71 0)
 			(effects
